Commit message: added transmission code to xacro file

File: src/robotic-arm-urdf-min/urdf/robotic-arm-urdf-min.urdf.xacro (robot description, xacro)
@@ -1,4 +1,8 @@
 <?xml version="1.0" encoding="utf-8"?>
 <robot name="robotic-arm-urdf-min">
+  <xacro:macro name="default_transmission" params="number">
+    <transmission>
+    </transmission>
+  </xacro:macro>
   <link name="base_link">
     <inertial>

Commit message: added control xacro

File: src/robotic-arm-urdf-min/urdf/robotic-arm-urdf-min.urdf.xacro (robot description, xacro)
@@ -1,6 +1,13 @@
 <?xml version="1.0" encoding="utf-8"?>
 <robot name="robotic-arm-urdf-min">
+  <xacro:include filename="$(find robotic-arm-urdf-min)/urdf/robotic-arm-gazebo.xacro" />
+  <xacro:include filename="$(find robotic-arm-urdf-min)/urdf/robotic-arm-control.xacro" />
   <xacro:macro name="default_transmission" params="number">
-    <transmission>
+    <transmission name="transmission_${number}">
+      <plugin>transmission_interface/SimpleTransmission</plugin>
+      <actuator name="actuator_${number}" role="actuator1" />
+      <joint name="joint_${number}" role="joint1">
+        <mechanical_reduction>1</mechanical_reduction>
+      </joint>
     </transmission>
   </xacro:macro>
@@ -230,3 +237,10 @@
     <limit lower="-3.14" upper="3.14" effort="300" velocity="3" />
   </joint>
+  <xacro:default_transmission number="1" />
+  <xacro:default_transmission number="2" />
+  <xacro:default_transmission number="3" />
+  <xacro:default_transmission number="4" />
+  <xacro:default_transmission number="5" />
+  <xacro:default_transmission number="6" />
+  <xacro:default_transmission number="7" />
 </robot>
