Commit message: working moveit and rviz gui

File: src/robotic-arm-urdf-min/urdf/robotic-arm-control.xacro (robot description, xacro)
@@ -1,4 +1,5 @@
-<?xml version="1.0"?>
-<robot xmls:xacro="http://www.ros.org/wiki/xacro" name="robotic-arm-urdf-min">
+<?xml version="1.0" encoding="utf-8"?>
+<robot name="robotic-arm-urdf-min"
+    xmlns:xacro="http://www.ros.org/wiki/xacro">
     <xacro:property name="PI" value="3.14159" />
     <ros2_control name="RobotSystem" type="system">

File: src/robotic-arm-urdf-min/urdf/robotic-arm-gazebo.xacro (robot description, xacro)
@@ -6,5 +6,5 @@
         <robot_param>robot_description</robot_param>
         <robot_param_node>robot_state_publisher</robot_param_node>
-        <parameters>$(find robot_arm_controller_test)/config/robot_controller.yaml</parameters>
+        <parameters>$(find moveit_config)/config/ros2_controllers.yaml</parameters>
     </gazebo>
 </robot>

File: src/robotic-arm-urdf-min/urdf/robotic-arm-urdf-min-v2.urdf.xacro (robot description, xacro)
@@ -2,4 +2,9 @@
 <robot name="robotic-arm-urdf-min"
   xmlns:xacro="https://www.ros.org/wiki/xacro">
+  <link name="world"/>
+  <joint name="world_to_base" type="fixed">
+    <parent link="world"/>
+    <child link="base_link"/>
+  </joint>
   <link name="base_link">
     <inertial>

File: src/robotic-arm-urdf-min/urdf/robotic-arm-urdf-min.urdf.xacro (robot description, xacro)
@@ -1,4 +1,5 @@
 <?xml version="1.0" encoding="utf-8"?>
-<robot name="robotic-arm-urdf-min">
+<robot name="robotic-arm-urdf-min"
+  xmlns:xacro="http://www.ros.org/wiki/xacro">
   <xacro:include filename="$(find robotic-arm-urdf-min)/urdf/robotic-arm-gazebo.xacro" />
   <xacro:include filename="$(find robotic-arm-urdf-min)/urdf/robotic-arm-control.xacro" />
