Commit message: pushing before things might break

File: src/urdf_viz/urdf/urdf_viz.urdf (robot description, URDF)
Before this commit: robot urdf_viz, 10 links, 9 joints
Links:
- added link world
Joints:
- added joint world_to_base: type fixed, parent world, child base_link, origin xyz=0 0 0 rpy=0 0 0

File: src/urdf_viz/urdf/urdf_viz.urdf.xacro (robot description, xacro)
@@ -5,4 +5,10 @@
 <robot name="urdf_viz"
   xmlns:xacro="https://www.ros.org/wiki/xacro">
+  <link name="world" />
+  <joint name="world_to_base" type="fixed">
+    <parent link="world" />
+    <child link="base_link" />
+    <origin xyz="0 0 0" rpy="0 0 0" />
+  </joint>
   <link name="base_link">
     <inertial>
