Commit message: first push to the new branch, updated urdf

File: src/arm_description/urdf/arm_description.urdf (robot description, URDF)
Before this commit: robot arm_description, 12 links, 11 joints
Links:
- removed link grip_left
- removed link grip_right
- removed link tool_frame
- added link grip_left_link, mass 0.0199960953484895; collision mesh filename=package://arm_description/meshes/grip_left_link.STL; visual mesh filename=package://arm_description/meshes/grip_left_link.STL
- added link grip_right_link, mass 0.0199960953484896; collision mesh filename=package://arm_description/meshes/grip_right_link.STL; visual mesh filename=package://arm_description/meshes/grip_right_link.STL
- added link tool_link, mass 0.125010719073419; collision mesh filename=package://arm_description/meshes/tool_link.STL; visual mesh filename=package://arm_description/meshes/tool_link.STL
- link base_link: mass 0.226867575584474 -> 0.244019918751533
Joints:
- removed joint grip_left
- removed joint grip_right
- added joint grip_left_join: type prismatic, parent tool_link, child grip_left_link, origin xyz=0 0 -0.119985205862429 rpy=0 0 0, axis -1 0 0, limit lower=-0.04 upper=0 effort=1 velocity=5
- added joint grip_right_joint: type prismatic, parent tool_link, child grip_right_link, origin xyz=0 0 -0.119985205862429 rpy=0 0 0, axis -1 0 0, limit lower=0 upper=0.04 effort=1 velocity=5
- joint joint_1: limit lower=-0.785398 upper=3.92699 effort=2 velocity=3 -> lower=-1.57 upper=3.14 effort=200 velocity=10
- joint joint_2: limit lower=-1.57 upper=1.57 effort=2 velocity=3 -> lower=-1.57 upper=1.57 effort=200 velocity=10
- joint joint_3: limit lower=-3.14 upper=3.14 effort=2 velocity=3 -> lower=-3.14 upper=3.14 effort=200 velocity=10
- joint joint_4: limit lower=-2.09 upper=2.09 effort=2 velocity=3 -> lower=-2.09 upper=2.09 effort=200 velocity=10
- joint joint_5: limit lower=-3.14 upper=3.14 effort=2 velocity=3 -> lower=-3.14 upper=3.14 effort=200 velocity=10
- joint joint_6: limit lower=-2.09 upper=2.09 effort=2 velocity=3 -> lower=-2.09 upper=2.09 effort=200 velocity=10
- joint joint_7: limit lower=-2.09 upper=2.09 effort=2 velocity=3 -> lower=-3.14 upper=3.14 effort=200 velocity=10
- joint tool_joint: child tool_frame -> tool_link; limit lower=-2.09 upper=2.09 effort=2 velocity=3 -> lower=-3.14 upper=3.14 effort=200 velocity=5; origin xyz=0 -0.102485205862441 -0.0909852058624315 rpy=-1.5707963267949 0 0 -> xyz=0 0 -0.090985 rpy=-1.5708 0 0

File: src/arm_moveit/config/arm_description.ros2_control.xacro (robot description, xacro)
@@ -72,17 +72,17 @@
                 <state_interface name="velocity"/>
             </joint>
-            <joint name="grip_left">
+            <joint name="grip_left_join">
                 <command_interface name="position"/>
                 <command_interface name="velocity"/>
                 <state_interface name="position">
-                  <param name="initial_value">${initial_positions['grip_left']}</param>
+                  <param name="initial_value">${initial_positions['grip_left_join']}</param>
                 </state_interface>
                 <state_interface name="velocity"/>
             </joint>
-            <joint name="grip_right">
+            <joint name="grip_right_joint">
                 <command_interface name="position"/>
                 <command_interface name="velocity"/>
                 <state_interface name="position">
-                  <param name="initial_value">${initial_positions['grip_right']}</param>
+                  <param name="initial_value">${initial_positions['grip_right_joint']}</param>
                 </state_interface>
                 <state_interface name="velocity"/>

Commit message: fixed gripper joint typo and added new rsp_controller pkg

File: src/arm_description/urdf/arm_description.urdf (robot description, URDF)
Before this commit: robot arm_description, 12 links, 11 joints
Joints:
- removed joint grip_left_join
- added joint grip_left_joint: type prismatic, parent tool_link, child grip_left_link, origin xyz=0 0 -0.119985205862429 rpy=0 0 0, axis -1 0 0, limit lower=-0.04 upper=0 effort=1 velocity=5

File: src/arm_moveit/config/arm_description.ros2_control.xacro (robot description, xacro)
@@ -72,9 +72,9 @@
                 <state_interface name="velocity"/>
             </joint>
-            <joint name="grip_left_join">
+            <joint name="grip_left_joint">
                 <command_interface name="position"/>
                 <command_interface name="velocity"/>
                 <state_interface name="position">
-                  <param name="initial_value">${initial_positions['grip_left_join']}</param>
+                  <param name="initial_value">${initial_positions['grip_left_joint']}</param>
                 </state_interface>
                 <state_interface name="velocity"/>

Commit message: new urdf with camera link working af, updated the path planning algorithm for drawing mode

File: src/arm_description/urdf/arm_description.urdf (robot description, URDF)
Before this commit: robot arm_description, 12 links, 11 joints
Links:
- added link cam_link, mass 0.0659679326018229; collision mesh filename=package://arm_description/meshes/cam_link.STL; visual mesh filename=package://arm_description/meshes/cam_link.STL
- link base_link: mass 0.244019918751533 -> 6.52720522593112
Joints:
- added joint cam_joint: type fixed, parent tool_link, child cam_link, origin xyz=0 0 -0.0135 rpy=0 0 0, axis 0 0 0
- joint grip_left_joint: origin xyz=0 0 -0.119985205862429 rpy=0 0 0 -> xyz=0 0 -0.0135 rpy=0 0 0
- joint grip_right_joint: origin xyz=0 0 -0.119985205862429 rpy=0 0 0 -> xyz=0 0 -0.0135 rpy=0 0 0
- joint tool_joint: origin xyz=0 0 -0.090985 rpy=-1.5708 0 0 -> xyz=0 -0.106485205862441 -0.0909852058624315 rpy=-1.5707963267949 0 0
